File: PCB/eChook Wireless Board/eChook Wireless Board.kicad_sch (KiCad schematic)
At the start: 31 parts, among them J1 POWER_CONNECTION, J10 WHEEL_RPM_CONNECTION, J11 5V_CONN, J12 STATUS_CONNECTION, J13 CURRENT_CONN, J14 TEMP_CONNECTION, J15 WHEEL_CONN, J16 Screw_Terminal_01x06, J17 Screw_Terminal_01x06, J2 POWER_SWITCH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

Commit message: Updated wireless board to V1.1
Fixed unconnected ground plane error of V1.0 board.
Parts:
- removed SW1: SW_DIP_x02, Button_Switch_THT:SW_DIP_SPSTx02_Slide_9.78x7.26mm_W7.62mm_P2.54mm, symbol Switch:SW_DIP_x02
- added J18: STATUS_CONNECTION, Connector_JST:JST_XH_B3B-XH-A_1x03_P2.50mm_Vertical, symbol SparkFun-Connectors:CONN_03JST-PTH
- J16, J17: footprint Connectors:SCREWTERMINAL-3.5MM-6 -> (none)
Connections:
- net GND: now also J18.3
- net DEBUG_MODE renamed MODE_INPUT_1
- net MODE_INPUT_1: now also J18.1
- net F24_MODE renamed MODE_INPUT_2
- net MODE_INPUT_2: now also J18.2
